Commit message: m2wr.launch added

File: src/m2wr_description/urdf/m2wr.xacro (robot description, xacro)
@@ -150,22 +150,2 @@
   </joint>
 </robot>
-1
-2
-3
-4
-5
-6
-7
-8
-9
-10
-<?xml version="1.0" ?>
-<robot name="m2wr" xmlns:xacro="http://www.ros.org/wiki/xacro">
-  <material name="black">
-    <color rgba="0.0 0.0 0.0 1.0"/>
-  </material>
-  <material name="blue">
-    <color rgba="0.203125 0.23828125 0.28515625 1.0"/>
-  </material>
-  <material name="green">
-    <color rgba="0.0 0.8 0.0 1.0"/>
